File: Hardware/Buck5V/SparkFun_Buck_Regulator_AP63357DV-7_Buck5V.brd (EAGLE design)
At the start: 25.4 x 25.4 mm, 49 parts, among them J3 POWER_JACK, U1 AP63357

Commit message: Added BabyBuck design.
Parts:
- added U$21: (no value), output:#GND#1
- added U$22: (no value), SparkFun-Aesthetics:HIGH_TEMP_WARNING
- added U$23: (no value), SparkFun-Aesthetics:ORDERING_INSTRUCTIONS
- moved U$20 3.58 mm to (18.4, 0.89)
- moved R5 1.69 mm to (16.1, 1.52), turned to 270 degrees
- moved D1 1.20 mm to (18.2, 2.03)
- moved U$1 0.38 mm to (10.7, 1.91)
- moved U$2 0.38 mm to (10.7, 0.89)
Routing:
- net N$5: track 3.60 -> 6.93 mm
- net 5V: track 8.11 -> 6.01 mm
- net GND: track 1.28 -> 1.89 mm, vias 83 -> 81

Commit message: Added dimensions, ordering instructions, set board stackup.
Parts:
- moved U$23 8.49 mm to (35.6, 43.1)
- moved FRAME1 7.50 mm to (21.2, -16.4)
Other:
- board text added: "Board thickness is 0.8mm 4-Layer 1oz copper outer 1oz copper inner"
- board text added: "UNITS IN INCHES"
Changed lines of the file:
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@@
 <drawing>
 <settings>
-<setting alwaysvectorfont="yes"/>
+<setting alwaysvectorfont="no"/>
 <setting verticaltext="up"/>
 </settings>
@@
 <dimension x1="0" y1="0" x2="2.54" y2="2.54" x3="-0.635" y3="1.27" textsize="0.889" textratio="15" layer="47" dtype="vertical" unit="inch"/>
 <dimension x1="0" y1="0" x2="3.683" y2="17.78" x3="-3.175" y3="8.89" textsize="0.889" textratio="15" layer="47" dtype="vertical" unit="inch"/>
-<dimension x1="0" y1="0" x2="23.495" y2="17.78" x3="28.321" y3="8.89" textsize="0.889" textratio="15" layer="47" dtype="vertical" unit="inch"/>
 <dimension x1="0" y1="0" x2="2.54" y2="22.86" x3="-5.334" y3="11.43" textsize="0.889" textratio="15" layer="47" dtype="vertical" unit="inch"/>
 <dimension x1="0" y1="0" x2="0" y2="25.4" x3="-8.128" y3="12.7" textsize="0.889" textratio="15" layer="47" dtype="vertical" unit="inch"/>
-<text x="49.149" y="-8.89" size="1.778" layer="51" font="vector" ratio="15">Alex Brudner</text>
+<text x="48.768" y="-16.383" size="1.778" layer="51" font="vector" ratio="15">Alex Brudner</text>
 <wire x1="7.493" y1="14.653259375" x2="7.112" y2="14.272259375" width="0.2032" layer="21"/>
 <wire x1="7.112" y1="14.272259375" x2="7.7851" y2="14.272259375" width="0.2032" layer="21"/>
@@
 <wire x1="7.493" y1="11.097259375" x2="7.112" y2="10.716259375" width="0.2032" layer="21"/>
 <wire x1="7.112" y1="10.716259375" x2="7.493" y2="10.335259375" width="0.2032" layer="21"/>
+<dimension x1="0" y1="0" x2="12.827" y2="9.906" x3="6.4135" y3="-2.286" textsize="0.889" layer="47" dtype="horizontal" unit="inch"/>
+<dimension x1="0" y1="0" x2="12.827" y2="9.906" x3="27.178" y3="4.953" textsize="0.889" layer="47" dtype="vertical" unit="inch"/>
+<dimension x1="5.207" y1="16.256" x2="20.447" y2="16.256" x3="12.827" y3="-6.096" textsize="0.889" layer="47" unit="inch"/>
+<dimension x1="5.207" y1="16.256" x2="5.207" y2="3.556" x3="30.607" y3="9.906" textsize="0.889" layer="47" unit="inch"/>
+<dimension x1="0" y1="0" x2="23.495" y2="17.78" x3="32.258" y3="8.89" textsize="0.889" layer="47" dtype="vertical" unit="inch"/>
+<text x="37.338" y="22.479" size="1.778" layer="51" font="vector">Board thickness is 0.8mm
+4-Layer
+1oz copper outer
+1oz copper inner</text>
+<text x="6.731" y="43.815" size="1.016" layer="47" font="vector">UNITS IN INCHES</text>
+<wire x1="3.683" y1="17.78" x2="3.683" y2="7.239" width="4.5212" layer="48"/>
+<wire x1="3.683" y1="7.239" x2="0.635" y2="4.191" width="4.5212" layer="48"/>
 </plain>
 <attributes>
@@
 </class>
 </classes>
-<designrules name="SparkFun-4-Layer-Minimum-JLCPCB">
+<designrules name="SparkFun-4-Layer-Minimum-JLCPCB *">
 <description language="en">&lt;b&gt;4 Layer Minimum Rules for JLCPCB&lt;/b&gt;
 &lt;p&gt;
@@
 &lt;/ul&gt;</description>
 <param name="layerSetup" value="(1*2*15*16)"/>
-<param name="mtCopper" value="0.035559375mm 0.035559375mm 0.035mm 0.035mm 0.035mm 0.035mm 0.035mm 0.035mm 0.035mm 0.035mm 0.035mm 0.035mm 0.035mm 0.035mm 0.035559375mm 0.035559375mm"/>
-<param name="mtIsolate" value="0.47751875mm 0.47751875mm 0.2mm 0.15mm 0.2mm 0.15mm 0.2mm 0.15mm 0.2mm 0.15mm 0.2mm 0.15mm 0.2mm 0.15mm 0.47751875mm"/>
+<param name="mtCopper" value="0.035mm 0.035mm 0.035mm 0.035mm 0.035mm 0.035mm 0.035mm 0.035mm 0.035mm 0.035mm 0.035mm 0.035mm 0.035mm 0.035mm 0.035mm 0.035mm"/>
+<param name="mtIsolate" value="0.2104mm 0.24mm 0.2mm 0.15mm 0.2mm 0.15mm 0.2mm 0.15mm 0.2mm 0.15mm 0.2mm 0.15mm 0.2mm 0.15mm 0.2104mm"/>
 <param name="mdWireWire" value="5mil"/>
 <param name="mdWirePad" value="5mil"/>
@@
 </autorouter>
 <elements>
-<element name="FRAME1" library="SparkFun-Aesthetics" package="CREATIVE_COMMONS" value="FRAME-LEDGER" x="21.59" y="-8.89" smashed="yes">
-<attribute name="DESIGNER" value="Alex Brudner" x="21.59" y="-8.89" size="1.778" layer="27" display="off"/>
-<attribute name="REV" value="v01" x="21.59" y="-8.89" size="1.778" layer="27" display="off"/>
+<element name="FRAME1" library="SparkFun-Aesthetics" package="CREATIVE_COMMONS" value="FRAME-LEDGER" x="21.209" y="-16.383" smashed="yes">
+<attribute name="DESIGNER" value="Alex Brudner" x="21.209" y="-16.383" size="1.778" layer="27" display="off"/>
+<attribute name="REV" value="v01" x="21.209" y="-16.383" size="1.778" layer="27" display="off"/>
 </element>
 <element name="FD1" library="SparkFun-Aesthetics" package="FIDUCIAL-MICRO" value="FIDUCIALUFIDUCIAL" x="24.765" y="0.635" smashed="yes"/>
@@
 <element name="U$21" library="output" package="#GND#1" value="" x="9.11351875" y="11.129009375" smashed="yes"/>
 <element name="U$22" library="SparkFun-Aesthetics" package="HIGH_TEMP_WARNING" value="" x="18.161" y="4.445" smashed="yes"/>
-<element name="U$23" library="SparkFun-Aesthetics" package="ORDERING_INSTRUCTIONS" value="" x="32.385" y="50.927" smashed="yes"/>
+<element name="U$23" library="SparkFun-Aesthetics" package="ORDERING_INSTRUCTIONS" value="" x="35.56" y="43.053" smashed="yes"/>
 </elements>
 <signals>
@@
 </drawing>
 <compatibility>
+<note version="6.3" minversion="6.2.2" severity="warning">
+Since Version 6.2.2 text objects can contain more than one line,
+which will not be processed correctly with this version.
+</note>
 <note version="8.3" severity="warning">
 Since Version 8.3, EAGLE supports URNs for individual library
