File: Hardware/Buck5V/SparkFun_Buck_Regulator_AP63357DV-7_Buck5V.sch (EAGLE design)
At the start: 29 parts, among them J3 POWER_JACK, U1 AP63357

Commit message: Ready for v10 reds.
1x1 - Thicken silk border on U1
micro - Move fiducial to increase heat sink size
both - panelize
Parts:
- FRAME1: REV v01 -> v10
Changed lines of the file:
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@@
 <part name="FRAME1" library="SparkFun-Aesthetics" deviceset="FRAME-LEDGER" device="">
 <attribute name="DESIGNER" value="Alex Brudner"/>
-<attribute name="REV" value="v01"/>
+<attribute name="REV" value="v10"/>
 </part>
 <part name="FD1" library="SparkFun-Aesthetics" deviceset="FIDUCIAL" device="UFIDUCIAL"/>
