File: Production/Buck5V/Panel/SparkFun_Buck_Regulator_AP63357DV-7_Buck5V-Panel.brd (EAGLE design)
At the start: 175 x 117.3 mm, 1254 parts, among them J11 POWER_JACK, J14 POWER_JACK, J17 POWER_JACK, J20 POWER_JACK, J23 POWER_JACK, J26 POWER_JACK, J29 POWER_JACK, J3 POWER_JACK, J32 POWER_JACK, J35 POWER_JACK, J38 POWER_JACK, J41 POWER_JACK, J44 POWER_JACK, J47 POWER_JACK, J5 POWER_JACK, J50 POWER_JACK, J53 POWER_JACK, J56 POWER_JACK, J59 POWER_JACK, J62 POWER_JACK, J65 POWER_JACK, J68 POWER_JACK, J71 POWER_JACK, J8 POWER_JACK, U1 AP63357, U10 AP63357, U11 AP63357, U12 AP63357, U13 AP63357, U14 AP63357, U15 AP63357, U16 AP63357, U17 AP63357, U18 AP63357, U19 AP63357, U2 AP63357, U20 AP63357, U21 AP63357, U22 AP63357, U23 AP63357, U24 AP63357, U3 AP63357, U4 AP63357, U5 AP63357, U6 AP63357, U7 AP63357, U8 AP63357, U9 AP63357

Commit message: Prepare for v10 reds order.
Change R1/R2 to better match 5V output requirement.
Repanelize.
Reorganize Production Folder Structure.
Parts:
- R1: value 150k -> 220K
- R10, R100, R105, R110, R115, R120, R15, R20, R25, R30, R35, R40, R45, R50, R55, R60, R65, R70, R75, R80, R85, R90, R95: value 2.2k -> 220K
- R101, R106, R11, R111, R116, R16, R2, R21, R26, R31, R36, R41, R46, R51, R56, R6, R61, R66, R71, R76, R81, R86, R91, R96: value 28.7k -> 41.2K
- R102, R107, R112, R117, R12, R17, R22, R27, R32, R37, R42, R47, R52, R57, R62, R67, R7, R72, R77, R82, R87, R92, R97: value 150k -> 93.1k; device SparkFun-Resistors:0402-TIGHT -> Buck5V:0402-TIGHT
- R103, R108, R113, R118, R13, R18, R23, R28, R33, R38, R43, R48, R53, R58, R63, R68, R73, R78, R8, R83, R88, R93, R98: value 93.1k -> 22k; device Buck5V:0402-TIGHT -> SparkFun-Resistors:0402-TIGHT
- R104, R109, R114, R119, R14, R19, R24, R29, R34, R39, R44, R49, R54, R59, R64, R69, R74, R79, R84, R89, R9, R94, R99: value 22k -> 2.2k
- moved R59 15.3 mm to (145.7, 27.4), turned to 270 degrees
- moved R34 15.3 mm to (16.1, 27.4), turned to 270 degrees
- moved R39 15.3 mm to (42.0, 27.4), turned to 270 degrees
- moved R49 15.3 mm to (93.9, 27.4), turned to 270 degrees
- moved R54 15.3 mm to (119.8, 27.4), turned to 270 degrees
- moved R119 15.3 mm to (145.7, 79.2), turned to 270 degrees
- moved R29 15.3 mm to (145.7, 1.52), turned to 270 degrees
- moved R89 15.3 mm to (145.7, 53.3), turned to 270 degrees
- moved R109 15.3 mm to (93.9, 79.2), turned to 270 degrees
- moved R114 15.3 mm to (119.8, 79.2), turned to 270 degrees
- moved R19 15.3 mm to (93.9, 1.52), turned to 270 degrees
- moved R24 15.3 mm to (119.8, 1.52), turned to 270 degrees
- moved R44 15.3 mm to (67.9, 27.4), turned to 270 degrees
- moved R64 15.3 mm to (16.1, 53.3), turned to 270 degrees
- moved R69 15.3 mm to (42.0, 53.3), turned to 270 degrees
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Connections:
- net 5V1: now also R10.2; no longer R7.2
- net 5V10: now also R55.2; no longer R52.2
- net 5V11: now also R60.2; no longer R57.2
- net 5V12: now also R65.2; no longer R62.2
- net 5V13: now also R70.2; no longer R67.2
- net 5V14: now also R75.2; no longer R72.2
- net 5V15: now also R80.2; no longer R77.2
- net 5V16: now also R85.2; no longer R82.2
- net 5V17: now also R90.2; no longer R87.2
- net 5V18: now also R95.2; no longer R92.2
- net 5V19: now also R100.2; no longer R97.2
- net 5V2: now also R15.2; no longer R12.2
- net 5V20: now also R105.2; no longer R102.2
- net 5V21: now also R110.2; no longer R107.2
- net 5V22: now also R115.2; no longer R112.2
- net 5V23: now also R120.2; no longer R117.2
- net 5V3: now also R20.2; no longer R17.2
- net 5V4: now also R25.2; no longer R22.2
- net 5V5: now also R30.2; no longer R27.2
- net 5V6: now also R35.2; no longer R32.2
- net 5V7: now also R40.2; no longer R37.2
- net 5V8: now also R45.2; no longer R42.2
- net 5V9: now also R50.2; no longer R47.2
- net EN1: now also R7.1, R8.2; no longer R8.1, R9.2
- net EN10: now also R52.1, R53.2; no longer R53.1, R54.2
- net EN11: now also R57.1, R58.2; no longer R58.1, R59.2
- net EN12: now also R62.1, R63.2; no longer R63.1, R64.2
- net EN13: now also R67.1, R68.2; no longer R68.1, R69.2
- net EN14: now also R72.1, R73.2; no longer R73.1, R74.2
- net EN15: now also R77.1, R78.2; no longer R78.1, R79.2
- net EN16: now also R82.1, R83.2; no longer R83.1, R84.2
- net EN17: now also R87.1, R88.2; no longer R88.1, R89.2
- net EN18: now also R92.1, R93.2; no longer R93.1, R94.2
- net EN19: now also R97.1, R98.2; no longer R98.1, R99.2
- net EN2: now also R12.1, R13.2; no longer R13.1, R14.2
- net EN20: now also R102.1, R103.2; no longer R103.1, R104.2
- net EN21: now also R107.1, R108.2; no longer R108.1, R109.2
- net EN22: now also R112.1, R113.2; no longer R113.1, R114.2
- net EN23: now also R117.1, R118.2; no longer R118.1, R119.2
- net EN3: now also R17.1, R18.2; no longer R18.1, R19.2
- net EN4: now also R22.1, R23.2; no longer R23.1, R24.2
- net EN5: now also R27.1, R28.2; no longer R28.1, R29.2
- net EN6: now also R32.1, R33.2; no longer R33.1, R34.2
- net EN7: now also R37.1, R38.2; no longer R38.1, R39.2
- net EN8: now also R42.1, R43.2; no longer R43.1, R44.2
- net EN9: now also R47.1, R48.2; no longer R48.1, R49.2
- net FB1: now also R10.1; no longer R7.1
- net FB10: now also R55.1; no longer R52.1
- net FB11: now also R60.1; no longer R57.1
- net FB12: now also R65.1; no longer R62.1
- net FB13: now also R70.1; no longer R67.1
- net FB14: now also R75.1; no longer R72.1
- net FB15: now also R80.1; no longer R77.1
- net FB16: now also R85.1; no longer R82.1
- net FB17: now also R90.1; no longer R87.1
- net FB18: now also R95.1; no longer R92.1
- net FB19: now also R100.1; no longer R97.1
- net FB2: now also R15.1; no longer R12.1
- net FB20: now also R105.1; no longer R102.1
- net FB21: now also R110.1; no longer R107.1
- net FB22: now also R115.1; no longer R112.1
- net FB23: now also R120.1; no longer R117.1
- net FB3: now also R20.1; no longer R17.1
- net FB4: now also R25.1; no longer R22.1
- net FB5: now also R30.1; no longer R27.1
- net FB6: now also R35.1; no longer R32.1
- net FB7: now also R40.1; no longer R37.1
- net FB8: now also R45.1; no longer R42.1
- net FB9: now also R50.1; no longer R47.1
- net GND1: now also R8.1; no longer R9.1
- net GND10: now also R53.1; no longer R54.1
- net GND11: now also R58.1; no longer R59.1
- net GND12: now also R63.1; no longer R64.1
- net GND13: now also R68.1; no longer R69.1
- net GND14: now also R73.1; no longer R74.1
- net GND15: now also R78.1; no longer R79.1
- net GND16: now also R83.1; no longer R84.1
- net GND17: now also R88.1; no longer R89.1
- net GND18: now also R93.1; no longer R94.1
- net GND19: now also R98.1; no longer R99.1
- net GND2: now also R13.1; no longer R14.1
- net GND20: now also R103.1; no longer R104.1
- net GND21: now also R108.1; no longer R109.1
- net GND22: now also R113.1; no longer R114.1
- net GND23: now also R118.1; no longer R119.1
- net GND3: now also R18.1; no longer R19.1
- net GND4: now also R23.1; no longer R24.1
- net GND5: now also R28.1; no longer R29.1
- net GND6: now also R33.1; no longer R34.1
- net GND7: now also R38.1; no longer R39.1
- net GND8: now also R43.1; no longer R44.1
- net GND9: now also R48.1; no longer R49.1
- net N$11: now also R19.1; no longer R20.1
- net N$12: now also R19.2; no longer R20.2
- net N$14: now also R24.1; no longer R25.1
- net N$15: now also R24.2; no longer R25.2
- net N$17: now also R29.1; no longer R30.1
- net N$18: now also R29.2; no longer R30.2
- net N$20: now also R34.1; no longer R35.1
- net N$21: now also R34.2; no longer R35.2
- net N$23: now also R39.1; no longer R40.1
- net N$24: now also R39.2; no longer R40.2
- net N$26: now also R44.1; no longer R45.1
- net N$27: now also R44.2; no longer R45.2
- net N$29: now also R49.1; no longer R50.1
- net N$3: now also R9.1; no longer R10.1
- net N$30: now also R49.2; no longer R50.2
- net N$32: now also R54.1; no longer R55.1
- net N$33: now also R54.2; no longer R55.2
- net N$35: now also R59.1; no longer R60.1
- net N$36: now also R59.2; no longer R60.2
- net N$38: now also R64.1; no longer R65.1
- net N$39: now also R64.2; no longer R65.2
- net N$41: now also R69.1; no longer R70.1
- net N$42: now also R69.2; no longer R70.2
- net N$44: now also R74.1; no longer R75.1
- net N$45: now also R74.2; no longer R75.2
- net N$47: now also R79.1; no longer R80.1
- net N$48: now also R79.2; no longer R80.2
- net N$50: now also R84.1; no longer R85.1
- net N$51: now also R84.2; no longer R85.2
- net N$53: now also R89.1; no longer R90.1
- net N$54: now also R89.2; no longer R90.2
- net N$56: now also R94.1; no longer R95.1
- net N$57: now also R94.2; no longer R95.2
- net N$59: now also R99.1; no longer R100.1
- net N$6: now also R9.2; no longer R10.2
- net N$60: now also R99.2; no longer R100.2
- net N$62: now also R104.1; no longer R105.1
- net N$63: now also R104.2; no longer R105.2
- net N$65: now also R109.1; no longer R110.1
- net N$66: now also R109.2; no longer R110.2
- net N$68: now also R114.1; no longer R115.1
- net N$69: now also R114.2; no longer R115.2
- net N$71: now also R119.1; no longer R120.1
- net N$72: now also R119.2; no longer R120.2
- net N$8: now also R14.1; no longer R15.1
- net N$9: now also R14.2; no longer R15.2
- net VIN1: now also R7.2; no longer R8.2
- net VIN10: now also R52.2; no longer R53.2
- net VIN11: now also R57.2; no longer R58.2
- net VIN12: now also R62.2; no longer R63.2
- net VIN13: now also R67.2; no longer R68.2
- net VIN14: now also R72.2; no longer R73.2
- net VIN15: now also R77.2; no longer R78.2
- net VIN16: now also R82.2; no longer R83.2
- net VIN17: now also R87.2; no longer R88.2
- net VIN18: now also R92.2; no longer R93.2
- net VIN19: now also R97.2; no longer R98.2
- net VIN2: now also R12.2; no longer R13.2
- net VIN20: now also R102.2; no longer R103.2
- net VIN21: now also R107.2; no longer R108.2
- net VIN22: now also R112.2; no longer R113.2
- net VIN23: now also R117.2; no longer R118.2
- net VIN3: now also R17.2; no longer R18.2
- net VIN4: now also R22.2; no longer R23.2
- net VIN5: now also R27.2; no longer R28.2
- net VIN6: now also R32.2; no longer R33.2
- net VIN7: now also R37.2; no longer R38.2
- net VIN8: now also R42.2; no longer R43.2
- net VIN9: now also R47.2; no longer R48.2
